File: KiCad/ardATProgrammer/ardATProgrammer.kicad_sch (KiCad schematic)
At the start: 21 parts

Commit message: kicad7
Parts:
- C? (x2): value (none) -> 22p
- C? (x4): value (none) -> 100n
- C?: value (none) -> 10u
- D? (x2): value (none) -> LED
- J?: value (none) -> 6-pin_FTDI_header
- J?: value (none) -> 2x3_ISP_header
- J?: value (none) -> 2x5_ISP_header
- JP? (x2): value (none) -> Jumper
- R?: value (none) -> 10k
- R? (x2): value (none) -> 330R
- U?: value (none) -> ATtiny85-20PU; footprint (none) -> Package_DIP:DIP-8_W7.62mm
- U?: value (none) -> ATtiny2313-20PU; footprint (none) -> Package_DIP:DIP-20_W7.62mm
- U?: value (none) -> ATmega328P-PU; footprint (none) -> Package_DIP:DIP-28_W7.62mm
- Y?: value (none) -> 16MHz
