File: KiCad/ardAVRProgrammer/ardAVRProgrammer.kicad_sch (KiCad schematic)
At the start: 13 parts, among them J1 2x5_ISP_header, J2 2x3_ISP_header, U1 ATmega328P-PU, U2 ATtiny2313-20M, U3 ATtiny85-20P

Commit message: new PCB layout
Parts:
- J1: footprint My_Headers:2x5_ISP_header_large -> My_Misc:IDC-Header_2x05_P2.54mm_Vertical_large
- J2: footprint My_Headers:2x3_ISP_header_large -> My_Misc:IDC-Header_2x03_P2.54mm_Vertical large
- U3: footprint My_Misc:DIP-8_W7.62mm_large -> My_Misc:DIP-8_W7.62mm_Socket_w_dip_packet_LongPads
Changed lines of the file:
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@@
     (property "Reference" "J2" (id 0) (at 171.069 48.895 0))
     (property "Value" "2x3_ISP_header" (id 1) (at 171.069 51.2064 0))
-    (property "Footprint" "My_Headers:2x3_ISP_header_large" (id 2) (at 166.37 57.15 0)
+    (property "Footprint" "My_Misc:IDC-Header_2x03_P2.54mm_Vertical large" (id 2) (at 166.37 57.15 0)
       (effects (font (size 1.27 1.27)) hide)
     )
@@
     (property "Reference" "J1" (id 0) (at 133.096 43.815 0))
     (property "Value" "2x5_ISP_header" (id 1) (at 133.096 46.1264 0))
-    (property "Footprint" "My_Headers:2x5_ISP_header_large" (id 2) (at 127 54.61 0)
+    (property "Footprint" "My_Misc:IDC-Header_2x05_P2.54mm_Vertical_large" (id 2) (at 127 54.61 0)
       (effects (font (size 1.27 1.27)) hide)
     )
@@
       (effects (font (size 1.27 1.27)) (justify right))
     )
-    (property "Footprint" "My_Misc:DIP-8_W7.62mm_large" (id 2) (at 132.08 171.45 0)
+    (property "Footprint" "My_Misc:DIP-8_W7.62mm_Socket_w_dip_packet_LongPads" (id 2) (at 132.08 171.45 0)
       (effects (font (size 1.27 1.27) italic) hide)
     )
@@
     )
     (path "/00000000-0000-0000-0000-00005ff18c02"
-      (reference "J1") (unit 1) (value "2x5_ISP_header") (footprint "My_Headers:2x5_ISP_header_large")
+      (reference "J1") (unit 1) (value "2x5_ISP_header") (footprint "My_Misc:IDC-Header_2x05_P2.54mm_Vertical_large")
     )
     (path "/00000000-0000-0000-0000-00005ff17a88"
-      (reference "J2") (unit 1) (value "2x3_ISP_header") (footprint "My_Headers:2x3_ISP_header_large")
+      (reference "J2") (unit 1) (value "2x3_ISP_header") (footprint "My_Misc:IDC-Header_2x03_P2.54mm_Vertical large")
     )
     (path "/00000000-0000-0000-0000-00005ff8e072"
@@
     )
     (path "/42a4fe1b-8275-4752-a085-94f9c8faf684"
-      (reference "U3") (unit 1) (value "ATtiny85-20P") (footprint "My_Misc:DIP-8_W7.62mm_large")
-    )
-  )
+      (reference "U3") (unit 1) (value "ATtiny85-20P") (footprint "My_Misc:DIP-8_W7.62mm_Socket_w_dip_packet_LongPads")
+    )
+  )

Commit message: kicad
Other:
- title: (none) -> ardAVRProgrammer
Changed lines of the file:
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@@
 (kicad_sch (version 20211123) (generator eeschema)
   (paper "A4")
+  (title_block
+    (title "ardAVRProgrammer")
+    (date "2022-09-09")
+    (rev "0.2")
+  )
   (junction (at 111.76 71.12) (diameter 0) (color 0 0 0 0)
   )
